File: PCB/vmodvga.kicad_pcb (KiCad board)
At the start: 2 copper layers, 80 x 60.1 mm, 70 parts, among them J1 DE-15, J2 DE-15, J3 VHDCI, P1 50R, P2 50R, P3 50R, P4 50R, P5 CONN_1, P6 CONN_1, U1 ADP3303-3V3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

Commit message: VHDCI Connector footprint verified and GND plane added to top layer.
Routing:
- added copper zone on F.Cu, net /GND
Changed lines of the file:
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@@
   )
   (setup
-    (last_trace_width 0.13)
+    (last_trace_width 0.125)
     (user_trace_width 0.13)
     (user_trace_width 0.25)
@@
   (segment (start 94.27 70.71) (end 94.12 70.56) (width 0.13) (layer B.Cu) (net 23))
   (segment (start 92.97 70.92) (end 92.7 70.92) (width 0.13) (layer B.Cu) (net 23) (status 30))
-  (segment (start 93.9 87.32) (end 93.9 86.88) (width 0.13) (layer F.Cu) (net 24) (status C00000))
-  (segment (start 92.7 85.68) (end 92.7 85.32) (width 0.13) (layer F.Cu) (net 24) (status C00000))
-  (segment (start 93.9 86.88) (end 92.7 85.68) (width 0.13) (layer F.Cu) (net 24) (status C00000))
+  (segment (start 93.9 87.32) (end 93.9 86.88) (width 0.13) (layer F.Cu) (net 24))
+  (segment (start 92.7 85.68) (end 92.7 85.32) (width 0.13) (layer F.Cu) (net 24))
+  (segment (start 93.9 86.88) (end 92.7 85.68) (width 0.13) (layer F.Cu) (net 24))
   (segment (start 118.938 96.51) (end 118.45 96.51) (width 0.125) (layer B.Cu) (net 24))
   (segment (start 118.45 96.51) (end 118.42 96.48) (width 0.125) (layer B.Cu) (net 24))
@@
       )
     )
+  )
+  (zone (net 24) (net_name /GND) (layer F.Cu) (hatch edge 0.508)
+    (connect_pads (clearance 0.508))
+    (min_thickness 0.254)
+    (fill (arc_segments 16) (thermal_gap 0.508) (thermal_bridge_width 0.508))
+    (polygon
+      (pts
+        (xy 88.91 50.3) (xy 166.91 50.3) (xy 166.91 108.3) (xy 88.91 108.3)
+      )
+    )
