File: PCB/vmodvga.kicad_pcb (KiCad board)
At the start: 2 copper layers, 80 x 60.1 mm, 70 parts, among them J1 DE-15, J2 DE-15, J3 VHDCI, P1 50R, P2 50R, P3 50R, P4 50R, P5 CONN_1, P6 CONN_1, U1 ADP3303-3V3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

Commit message: GND plan changed
Routing:
- net /GND: track 138.1 -> 141.0 mm
